File: pcb/Project.kicad_pcb (KiCad board)
At the start: 2 copper layers, 80.1 x 76.4 mm, 27 parts, among them J1 Display, SW1 SW_Push, SW10 SW_Push, SW11 SW_Push, SW12 SW_Push, SW13 SW_Push, SW2 SW_Push, SW3 SW_Push, SW4 SW_Push, SW5 RotaryEncoder, SW6 SW_Push, SW7 SW_Push, SW8 SW_Push, SW9 SW_Push, U1 MOUDLE-SEEEDUINO-XIAO

Commit message: The Pain
Parts:
- D1, D12, D8: footprint Diode_SMD:D_SOD-523 -> Diode_THT:D_DO-35_SOD27_P7.62mm_Horizontal
- D10: renamed from D4; footprint Diode_SMD:D_SOD-523 -> Diode_THT:D_DO-35_SOD27_P7.62mm_Horizontal
- D11: renamed from D7; footprint Diode_SMD:D_SOD-523 -> Diode_THT:D_DO-35_SOD27_P7.62mm_Horizontal
- D2: renamed from D5; footprint Diode_SMD:D_SOD-523 -> Diode_THT:D_DO-35_SOD27_P7.62mm_Horizontal
- D3: renamed from D9; footprint Diode_SMD:D_SOD-523 -> Diode_THT:D_DO-35_SOD27_P7.62mm_Horizontal
- D4: renamed from D2; footprint Diode_SMD:D_SOD-523 -> Diode_THT:D_DO-35_SOD27_P7.62mm_Horizontal
- D5: renamed from D6; footprint Diode_SMD:D_SOD-523 -> Diode_THT:D_DO-35_SOD27_P7.62mm_Horizontal
- D6: renamed from D10; footprint Diode_SMD:D_SOD-523 -> Diode_THT:D_DO-35_SOD27_P7.62mm_Horizontal
- D7: renamed from D3; footprint Diode_SMD:D_SOD-523 -> Diode_THT:D_DO-35_SOD27_P7.62mm_Horizontal
- D9: renamed from D11; footprint Diode_SMD:D_SOD-523 -> Diode_THT:D_DO-35_SOD27_P7.62mm_Horizontal
- moved D7 7.67 mm to (143.4, 69.9), turned to 90 degrees
- moved D8 7.67 mm to (143.4, 89.0), turned to 90 degrees
- moved D9 7.67 mm to (143.4, 108.1), turned to 90 degrees
- moved D1 7.67 mm to (105.3, 70.0), turned to 90 degrees
- moved D2 7.67 mm to (105.3, 89.1), turned to 90 degrees
- moved D6 7.67 mm to (124.3, 108.0), turned to 90 degrees
- moved D10 7.67 mm to (162.5, 70.0), turned to 90 degrees
- moved D11 7.67 mm to (162.5, 89.0), turned to 90 degrees
- moved D12 7.67 mm to (162.4, 108.1), turned to 90 degrees
- moved D3 7.67 mm to (105.3, 108.1), turned to 90 degrees
- moved D4 7.67 mm to (124.4, 70.0), turned to 90 degrees
- moved D5 7.67 mm to (124.3, 89.0), turned to 90 degrees
- renumbered SW2 to SW1, SW4 to SW10, SW9 to SW11, SW13 to SW12, SW5 to SW13, SW7 to SW2, SW10 to SW3, SW1 to SW4, SW6 to SW5, SW11 to SW6, SW3 to SW7, SW12 to SW9
Connections:
- net +3V3 renamed Net-(J1-VCC)
- net /D0 renamed /ROW3
- net /D1 renamed /ROW2
- net /D10 renamed Net-(U1-PA6_A10_D10_MOSI)
- net /D2 renamed /ROW1
- net /D3 renamed /ROW0
- net /D9 renamed Net-(U1-PA5_A9_D9_MISO)
- J1 pad 1: GND -> /GND
- SW13 pad C: unconnected-(SW13-PadC) -> /GND
- U1 pad 13: GND -> /GND
- U1 pad 14: +5V -> unconnected-(U1-5V-Pad14)
Routing:
- net /ROW0: track 54.9 -> 71.9 mm
- net /ROW2: track 84.6 -> 98.3 mm
- net /ROW3: track 105.3 -> 118.6 mm
- net /ROW1: track 62.9 -> 76.0 mm
- net /GND: track 0.00 -> 8.18 mm, vias 0 -> 2
- net Net-(D5-A): track 3.34 -> 4.99 mm
- net Net-(D7-A): track 3.34 -> 4.93 mm
- net Net-(D10-A): track 3.36 -> 4.94 mm
- net Net-(D8-A): track 3.34 -> 4.91 mm
- net Net-(D11-A): track 3.35 -> 4.91 mm
- net Net-(D4-A): track 3.35 -> 4.79 mm
- net Net-(D2-A): track 3.41 -> 4.85 mm
- net Net-(D9-A): track 3.34 -> 4.78 mm
- net Net-(D6-A): track 3.34 -> 4.78 mm
- net Net-(D3-A): track 3.34 -> 4.78 mm
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- added copper zone on B.Cu, net /GND
- removed copper zone on B.Cu, net GND
Other:
- board size 80.1 x 76.4 mm -> 80.1 x 76.5 mm
