File: pcb/Project.kicad_sch (KiCad schematic)
At the start: 27 parts, among them J1 Display, SW1 SW_Push, SW10 SW_Push, SW11 SW_Push, SW12 SW_Push, SW13 RotaryEncoder, SW2 SW_Push, SW3 SW_Push, SW4 SW_Push, SW5 SW_Push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

Commit message: The Pain
Parts:
- D1, D10, D11, D12, D2, D3, D4, D5, D6, D7, D8, D9: footprint Diode_SMD:D_SOD-523 -> Diode_THT:D_DO-35_SOD27_P7.62mm_Horizontal
Connections:
- net GND: now also SW13.C
- net +3V3: no longer names the net of J1.2 (VCC), U1.12 (3V3)
- net +5V: no longer names the net of U1.14 (5V)
- net D0 renamed ROW3
- net D1 renamed ROW2
- net D10: no longer names the net of SW13.A, U1.11 (PA6_A10_D10_MOSI)
- net D2 renamed ROW1
- net D3 renamed ROW0
- net D9: no longer names the net of SW13.B, U1.10 (PA5_A9_D9_MISO)
- no-connect marks 0 -> 1
